File: PCB/EPD75/EPD75.kicad_sch (KiCad schematic)
At the start: 35 parts, among them J1 Conn_01x26, J2 Shelly, J3 USB-PROG, Q1 DMG1012T, U2 ESP32-S3-MINI-1, U3 MD8942

Commit message: Started, but need a face up sockedt
Parts:
- J1: footprint RevK:24_Pins_0.5mm_Pitch_ZIF_Connector_UP -> RevK:HRS-FH12-24S-0.5SH-Face-Down; JLCPCB Rotation Offset 180 -> (none)
Connections:
- net BUSY: now also U2.34 (GPIO38)
- net CLK: now also U2.29 (GPIO34)
- net CS: now also U2.31 (GPIO35)
- net D+: now also U2.24 (GPIO20)
- net D-: now also U2.23 (GPIO19)
- net DC: now also U2.32 (GPIO36)
- net MOSI: now also U2.28 (GPIO33)
- net RST: now also U2.33 (GPIO37)
- no-connect marks 27 -> 24
Other:
- note added: "Find Face up socket"
- note removed: "CHECK FOOTPRINT CHECK POSITION"
Changed lines of the file:
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@@
   (no_connect (at 48.895 63.5))
   (no_connect (at 133.985 132.08))
-  (no_connect (at 79.375 71.12))
   (no_connect (at 48.895 60.96))
   (no_connect (at 79.375 91.44))
+  (no_connect (at 79.375 99.06))
+  (no_connect (at 79.375 96.52))
   (no_connect (at 48.895 58.42))
   (no_connect (at 153.035 45.72))
   (no_connect (at 48.895 50.8))
-  (no_connect (at 79.375 68.58))
   (no_connect (at 48.895 53.34))
   (no_connect (at 48.895 71.12))
@@
   (no_connect (at 79.375 86.36))
   (no_connect (at 133.985 147.32))
-  (no_connect (at 79.375 76.2))
   (no_connect (at 48.895 68.58))
   (no_connect (at 79.375 83.82))
@@
   (no_connect (at 79.375 93.98))
   (no_connect (at 79.375 81.28))
-  (no_connect (at 79.375 73.66))
-  (no_connect (at 79.375 63.5))
   (no_connect (at 48.895 73.66))
   (wire (pts (xy 160.655 109.22) (xy 172.085 109.22))
@@
     (effects (font (size 5 5)) (justify right bottom))
   )
+  (text "Find Face up socket" (at 98.425 177.8 0)
+    (effects (font (size 5 5)) (justify right bottom))
+  )
   (text "BELL PUSH - BAV99?" (at 104.775 130.81 0)
     (effects (font (size 5 5)) (justify right bottom))
-  )
-  (text "CHECK FOOTPRINT\nCHECK POSITION" (at 126.365 147.955 90)
-    (effects (font (size 5 5)) (justify left bottom))
   )
   (global_label "CLK" (shape input) (at 137.16 116.84 0) (fields_autoplaced)
@@
     )
   )
+  (global_label "MOSI" (shape output) (at 79.375 63.5 0) (fields_autoplaced)
+    (effects (font (size 1.27 1.27)) (justify left))
+    (property "Intersheetrefs" "${INTERSHEET_REFS}" (at 86.3022 63.5 0)
+      (effects (font (size 1.27 1.27)) (justify left) hide)
+    )
+  )
   (global_label "DC" (shape output) (at 103.505 49.53 0) (fields_autoplaced)
     (effects (font (size 1.27 1.27)) (justify left))
@@
     )
   )
+  (global_label "BUSY" (shape output) (at 79.375 76.2 0) (fields_autoplaced)
+    (effects (font (size 1.27 1.27)) (justify left))
+    (property "Intersheetrefs" "${INTERSHEET_REFS}" (at 86.6046 76.2 0)
+      (effects (font (size 1.27 1.27)) (justify left) hide)
+    )
+  )
   (global_label "DC" (shape input) (at 153.035 34.925 180) (fields_autoplaced)
     (effects (font (size 1.27 1.27)) (justify right))
@@
     )
   )
+  (global_label "DC" (shape output) (at 79.375 71.12 0) (fields_autoplaced)
+    (effects (font (size 1.27 1.27)) (justify left))
+    (property "Intersheetrefs" "${INTERSHEET_REFS}" (at 84.246 71.12 0)
+      (effects (font (size 1.27 1.27)) (justify left) hide)
+    )
+  )
   (global_label "CS" (shape input) (at 137.16 119.38 0) (fields_autoplaced)
     (effects (font (size 1.27 1.27)) (justify left))
@@
     )
   )
+  (global_label "D+" (shape bidirectional) (at 48.895 96.52 180) (fields_autoplaced)
+    (effects (font (size 1.27 1.27)) (justify right))
+    (property "Intersheetrefs" "${INTERSHEET_REFS}" (at 42.7691 96.52 0)
+      (effects (font (size 1.27 1.27)) (justify right) hide)
+    )
+  )
+  (global_label "RST" (shape output) (at 79.375 73.66 0) (fields_autoplaced)
+    (effects (font (size 1.27 1.27)) (justify left))
+    (property "Intersheetrefs" "${INTERSHEET_REFS}" (at 85.1531 73.66 0)
+      (effects (font (size 1.27 1.27)) (justify left) hide)
+    )
+  )
+  (global_label "CS" (shape output) (at 79.375 68.58 0) (fields_autoplaced)
+    (effects (font (size 1.27 1.27)) (justify left))
+    (property "Intersheetrefs" "${INTERSHEET_REFS}" (at 84.1855 68.58 0)
+      (effects (font (size 1.27 1.27)) (justify left) hide)
+    )
+  )
+  (global_label "D-" (shape bidirectional) (at 48.895 93.98 180) (fields_autoplaced)
+    (effects (font (size 1.27 1.27)) (justify right))
+    (property "Intersheetrefs" "${INTERSHEET_REFS}" (at 42.7691 93.98 0)
+      (effects (font (size 1.27 1.27)) (justify right) hide)
+    )
+  )
   (global_label "MOSI" (shape input) (at 137.16 114.3 0) (fields_autoplaced)
     (effects (font (size 1.27 1.27)) (justify left))
@@
     (effects (font (size 1.27 1.27)) (justify left))
     (property "Intersheetrefs" "${INTERSHEET_REFS}" (at 109.6309 56.515 0)
+      (effects (font (size 1.27 1.27)) (justify left) hide)
+    )
+  )
+  (global_label "CLK" (shape output) (at 79.375 66.04 0) (fields_autoplaced)
+    (effects (font (size 1.27 1.27)) (justify left))
+    (property "Intersheetrefs" "${INTERSHEET_REFS}" (at 85.2741 66.04 0)
       (effects (font (size 1.27 1.27)) (justify left) hide)
     )
@@
       (effects (font (size 1.27 1.27)) (justify left))
     )
-    (property "Footprint" "RevK:24_Pins_0.5mm_Pitch_ZIF_Connector_UP" (at 128.905 116.84 0)
+    (property "Footprint" "RevK:HRS-FH12-24S-0.5SH-Face-Down" (at 128.905 116.84 0)
       (effects (font (size 1.27 1.27)) hide)
     )
@@
       (effects (font (size 1.27 1.27)) hide)
     )
-    (property "JLCPCB Rotation Offset" "180" (at 128.905 116.84 0)
-      (effects (font (size 1.27 1.27)) hide)
-    )

Commit message: Better connector
Parts:
- J1: footprint RevK:HRS-FH12-24S-0.5SH-Face-Down -> RevK:XUNPU-FPC-05FB-24PH20; LCSC Part # C202112 -> C2856831
Changed lines of the file:
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@@
       (effects (font (size 1.27 1.27)) (justify left))
     )
-    (property "Footprint" "RevK:HRS-FH12-24S-0.5SH-Face-Down" (at 128.905 116.84 0)
+    (property "Footprint" "RevK:XUNPU-FPC-05FB-24PH20" (at 128.905 116.84 0)
       (effects (font (size 1.27 1.27)) hide)
     )
@@
       (effects (font (size 1.27 1.27)) hide)
     )
-    (property "LCSC Part #" "C202112" (at 128.905 116.84 0)
+    (property "LCSC Part #" "C2856831" (at 128.905 116.84 0)
       (effects (font (size 1.27 1.27)) hide)
     )

Commit message: Needs tracking
Parts:
- added C3: 0.1uF, RevK:C_0402, symbol Device:C
- added C5 (x4): 100nF, RevK:C_0402, symbol Device:C
- added C7, C8: 33pF, RevK:C_0402, symbol Device:C
- added D1, D2, D6, D7: XL-1010RGBC-WS2812B, RevK:SMD1010, symbol RevK:WS2812B-1mm
- added D4: BAV99S, RevK:SOT-363_SC-70-6, symbol Diode:BAV99S
- added D8: D, RevK:D_SOD-123, symbol Device:D
- added J4: BTN1, RevK:PTSM-HH-2-RA-SMD, symbol Connector_Generic:Conn_01x02
- added J5, J7: USB-C-Socket-V, RevK:USB-C-Socket-H, symbol RevK:USB-C-Socket-H
- added J6: BTN2, RevK:PTSM-HH-2-RA-SMD, symbol Connector_Generic:Conn_01x02
- added J8: PWR, RevK:PTSM-HH-2-RA-SMD, symbol Connector_Generic:Conn_01x02
- added JP1, JP2: SolderJumper_3_Bridged12, RevK:SolderJumper3, symbol Jumper:SolderJumper_3_Bridged12
- added P41, P42, P45: -, RevK:SolderPad, symbol RevK:SolderPad
- added P43: GND, RevK:SolderPad, symbol RevK:SolderPad
- added P43 (x2): 2, RevK:SolderPad, symbol RevK:SolderPad
- added P44 (x2): 1, RevK:SolderPad, symbol RevK:SolderPad
- added P44, P45, P46: +, RevK:SolderPad, symbol RevK:SolderPad
- added P46: 5V, RevK:SolderPad, symbol RevK:SolderPad
- added R1: 3R, RevK:R_0402, symbol Device:R
- added R12, R13: 100R, RevK:R_0402, symbol Device:R
- added R2 (x2), R3 (x2): 5k1, RevK:R_0402, symbol Device:R
- C3: value 4.7uF -> 10uF
Connections:
- net +3.3V: now also C3.1, C5.1, C5.1, C5.1, C5.1, D1.2 (+), D2.2 (+), D4.2 (K2), D4.5 (K4), D6.2 (+), D7.2 (+), JP1.3 (B)
- net BUSY: now also U2.31 (GPIO35); no longer U2.34 (GPIO38)
- net CLK: now also U2.35 (GPIO39); no longer U2.29 (GPIO34)
- net CS: now also U2.34 (GPIO38); no longer U2.31 (GPIO35)
- net D+: now also J5.A6 (D+), J5.B6 (D+), J7.A6 (D+), J7.B6 (D+), P44.1 (P)
- net D-: now also J5.A7 (D-), J5.B7 (D-), J7.A7 (D-), J7.B7 (D-), P45.1 (P)
- net DC: now also U2.33 (GPIO37); no longer J3.1 (VBUS), U2.32 (GPIO36), U3.5 (VIN)
- net GND: now also R1.1, C3.2, C5.2, C5.2, C5.2, C5.2, C7.2, C8.2, D1.3 (-), D2.3 (-), D4.1 (A1), D4.4 (A3), D6.3 (-), D7.3 (-), J4.1 (Pin_1), J5.A1 (GND), J5.A12 (GND), J5.B1 (GND), J5.B12 (GND), J5.S1 (SHIELD), J6.1 (Pin_1), J7.A1 (GND), J7.A12 (GND), J7.B1 (GND), J7.B12 (GND), J7.S1 (SHIELD), J8.1 (Pin_1), JP1.1 (A), P41.1 (P), P42.1 (P), P43.1 (P), P43.1 (P), P44.1 (P), R1.1, R2.2, R2.2, R3.2, R3.2; no longer J1.8 (Pin_8), R1.2, U2.16 (GPIO12), U2.17 (GPIO13), U2.18 (GPIO14), U2.19 (GPIO15), U2.20 (GPIO16), U2.21 (GPIO17), U2.22 (GPIO18)
- net MOSI: now also U2.36 (GPIO40); no longer U2.28 (GPIO33)
- net RST: now also U2.32 (GPIO36); no longer U2.33 (GPIO37)
- net at J1.2 (Pin_2), Q1.1 (G): now also R1.2; no longer R1.1
- net at J1.3 (Pin_3), Q1.2 (S): now also JP2.2 (C); no longer R1.1
- net BTN1: now reaches U2.37 (GPIO41)
- net BTN1: now also C8.1, D4.3 (K1A2), R13.2
- net BTN2: now reaches U2.38 (GPIO42)
- net BTN2: now also C7.1, D4.6 (K3A4), R12.2
- new net: D6.1 (O), D7.4 (I)
- new net: D2.1 (O), D6.4 (I)
- new net: J4.2 (Pin_2), P43.1 (P), R12.1
- new net: J6.2 (Pin_2), P44.1 (P), R13.1
- new net: D1.1 (O), D2.4 (I)
- new net: JP2.1 (A), R1.1
- new net: JP2.3 (B), R1.2
- new net: J5.A5 (CC1), R2.1
- new net: J5.B5 (CC2), R3.1
- new net: J7.A5 (CC1), R2.1
- new net: J7.B5 (CC2), R3.1
- new net: J1.8 (Pin_8), JP1.2 (C)
- new net PWR: D8.1 (K), J8.2 (Pin_2), P45.1 (P), P46.1 (P), U3.5 (VIN)
- new net RGB: D1.4 (I), U2.29 (GPIO34)
- new net VBUS: D8.2 (A), J3.1 (VBUS), J5.A4 (VBUS), J5.A9 (VBUS), J5.B4 (VBUS), J5.B9 (VBUS), J7.A4 (VBUS), J7.A9 (VBUS), J7.B4 (VBUS), J7.B9 (VBUS), P46.1 (P)
- no-connect marks 24 -> 29
Other:
- note removed: "12V power with big holes"
- note removed: "BELL PUSH - BAV99?"
- note removed: "Find Face up socket"
- note removed: "RECHECK E-PAPER CIRCUIT"
- moved on the sheet: C3, D1, D2, D3, J1, L1, Q1, R1

Commit message: Initial tracking
Parts:
- removed C3: 0.1uF, RevK:C_0402, symbol Device:C
Connections:
- net at P43.1 (P), R12.1: now also J6.2 (Pin_2); no longer J4.2 (Pin_2)
- net at P44.1 (P), R13.1: now also J4.2 (Pin_2); no longer J6.2 (Pin_2)
Other:
- moved on the sheet: J4, J6
Changed lines of the file:
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@@
     (comment 2 "www.me.uk")
   )
-  (junction (at 255.27 29.845) (diameter 0) (color 0 0 0 0)
-  )
   (junction (at 250.825 45.085) (diameter 0) (color 0 0 0 0)
   )
-  (junction (at 255.27 45.085) (diameter 0) (color 0 0 0 0)
-  )
   (junction (at 132.715 111.125) (diameter 0) (color 0 0 0 0)
   )
@@
   (junction (at 157.48 139.065) (diameter 0) (color 0 0 0 0)
   )
-  (junction (at 157.48 111.125) (diameter 0) (color 0 0 0 0)
-  )
   (junction (at 127.635 90.805) (diameter 0) (color 0 0 0 0)
   )
@@
   (junction (at 122.555 111.125) (diameter 0) (color 0 0 0 0)
   )
-  (junction (at 137.16 111.125) (diameter 0) (color 0 0 0 0)
-  )
   (junction (at 157.48 98.425) (diameter 0) (color 0 0 0 0)
   )
@@
   (junction (at 208.915 60.325) (diameter 0) (color 0 0 0 0)
   )
+  (junction (at 255.27 45.085) (diameter 0) (color 0 0 0 0)
+  )
   (junction (at 250.825 29.845) (diameter 0) (color 0 0 0 0)
   )
+  (junction (at 255.27 29.845) (diameter 0) (color 0 0 0 0)
+  )
   (junction (at 157.48 100.965) (diameter 0) (color 0 0 0 0)
   )
@@
     (stroke (width 0) (type default))
   )
-  (wire (pts (xy 137.16 111.125) (xy 147.32 111.125))
-    (stroke (width 0) (type default))
-  )
   (wire (pts (xy 215.265 67.945) (xy 221.615 67.945))
     (stroke (width 0) (type default))
@@
     (stroke (width 0) (type default))
   )
-  (wire (pts (xy 157.48 111.125) (xy 157.48 108.585))
+  (wire (pts (xy 157.48 108.585) (xy 157.48 123.19))
     (stroke (width 0) (type default))
   )
@@
     (stroke (width 0) (type default))
   )
-  (wire (pts (xy 154.94 111.125) (xy 157.48 111.125))
-    (stroke (width 0) (type default))
-  )
   (wire (pts (xy 246.38 145.415) (xy 250.19 145.415))
     (stroke (width 0) (type default))
   )
-  (wire (pts (xy 157.48 111.125) (xy 157.48 123.19))
-    (stroke (width 0) (type default))
-  )
   (wire (pts (xy 157.48 136.525) (xy 157.48 139.065))
     (stroke (width 0) (type default))
@@
     )
   )
-  (symbol (lib_id "Connector_Generic:Conn_01x02") (at 260.35 45.085 0) (mirror x) (unit 1)
+  (symbol (lib_id "Connector_Generic:Conn_01x02") (at 260.35 29.845 0) (mirror x) (unit 1)
     (in_bom no) (on_board yes) (dnp no)
-    (property "Reference" "J6" (at 262.382 45.0271 0)
+    (property "Reference" "J6" (at 262.382 29.7871 0)
       (effects (font (size 1.27 1.27)) (justify left))
     )
-    (property "Value" "BTN2" (at 262.382 42.6029 0)
+    (property "Value" "BTN2" (at 262.382 27.3629 0)
       (effects (font (size 1.27 1.27)) (justify left))
     )
-    (property "Footprint" "RevK:PTSM-HH-2-RA-SMD" (at 260.35 45.085 0)
+    (property "Footprint" "RevK:PTSM-HH-2-RA-SMD" (at 260.35 29.845 0)
       (effects (font (size 1.27 1.27)) hide)
     )
-    (property "Datasheet" "~" (at 260.35 45.085 0)
+    (property "Datasheet" "~" (at 260.35 29.845 0)
       (effects (font (size 1.27 1.27)) hide)
     )
@@
     )
   )
-  (symbol (lib_id "Device:C") (at 151.13 111.125 90) (unit 1)
-    (in_bom yes) (on_board yes) (dnp no)
-    (property "Reference" "C3" (at 147.32 109.855 90)
-      (effects (font (size 1.27 1.27)))
-    )
-    (property "Value" "0.1uF" (at 146.685 112.395 90)
-      (effects (font (size 1.27 1.27)))
-    )
-    (property "Footprint" "RevK:C_0402" (at 154.94 110.1598 0)
-      (effects (font (size 1.27 1.27)) hide)
-    )
-    (property "Datasheet" "~" (at 151.13 111.125 0)
-      (effects (font (size 1.27 1.27)) hide)
-    )
-    (pin "1")
-    (pin "2")
-    (instances
-      (project "USBA"
-        (path "/2d210a96-f81f-42a9-8bf4-1b43c11086f3"
-          (reference "C3") (unit 1)
-        )
-      )
-      (project "EPD75"
-        (path "/46c350bb-7de4-4e81-aafd-4af55e37aab0"
-          (reference "C23") (unit 1)
-        )
-      )
-    )
-  )
   (symbol (lib_id "Jumper:SolderJumper_3_Bridged12") (at 142.24 123.19 0) (mirror y) (unit 1)
     (in_bom no) (on_board yes) (dnp no)
@@
     )
   )
-  (symbol (lib_id "Connector_Generic:Conn_01x02") (at 260.35 29.845 0) (mirror x) (unit 1)
+  (symbol (lib_id "Connector_Generic:Conn_01x02") (at 260.35 45.085 0) (mirror x) (unit 1)
     (in_bom no) (on_board yes) (dnp no)
-    (property "Reference" "J4" (at 262.382 29.7871 0)
+    (property "Reference" "J4" (at 262.382 45.0271 0)
       (effects (font (size 1.27 1.27)) (justify left))
     )
-    (property "Value" "BTN1" (at 262.382 27.3629 0)
+    (property "Value" "BTN1" (at 262.382 42.6029 0)
       (effects (font (size 1.27 1.27)) (justify left))
     )
-    (property "Footprint" "RevK:PTSM-HH-2-RA-SMD" (at 260.35 29.845 0)
+    (property "Footprint" "RevK:PTSM-HH-2-RA-SMD" (at 260.35 45.085 0)
       (effects (font (size 1.27 1.27)) hide)
     )
-    (property "Datasheet" "~" (at 260.35 29.845 0)
+    (property "Datasheet" "~" (at 260.35 45.085 0)
       (effects (font (size 1.27 1.27)) hide)
     )

Commit message: 50V caps
Parts:
- C3: value 1uF -> 1uF 50V
- C3: value 100nF -> 100nF 50V
Other:
- moved on the sheet: C3
Changed lines of the file:
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@@
     (stroke (width 0) (type default))
   )
-  (wire (pts (xy 127.635 90.805) (xy 147.32 90.805))
+  (wire (pts (xy 127.635 90.805) (xy 148.59 90.805))
     (stroke (width 0) (type default))
   )
@@
     (stroke (width 0) (type default))
   )
-  (wire (pts (xy 154.94 100.965) (xy 157.48 100.965))
+  (wire (pts (xy 156.21 100.965) (xy 157.48 100.965))
     (stroke (width 0) (type default))
   )
@@
     (stroke (width 0) (type default))
   )
-  (wire (pts (xy 154.94 95.885) (xy 157.48 95.885))
+  (wire (pts (xy 156.21 95.885) (xy 157.48 95.885))
     (stroke (width 0) (type default))
   )
@@
     (stroke (width 0) (type default))
   )
-  (wire (pts (xy 129.54 95.885) (xy 147.32 95.885))
+  (wire (pts (xy 129.54 95.885) (xy 148.59 95.885))
     (stroke (width 0) (type default))
   )
@@
     (stroke (width 0) (type default))
   )
-  (wire (pts (xy 154.94 90.805) (xy 157.48 90.805))
+  (wire (pts (xy 156.21 90.805) (xy 157.48 90.805))
     (stroke (width 0) (type default))
   )
@@
     (stroke (width 0) (type default))
   )
-  (wire (pts (xy 119.38 100.965) (xy 147.32 100.965))
+  (wire (pts (xy 119.38 100.965) (xy 148.59 100.965))
     (stroke (width 0) (type default))
   )
@@
     )
   )
-  (symbol (lib_id "Device:C") (at 151.13 90.805 90) (unit 1)
+  (symbol (lib_id "Device:C") (at 152.4 90.805 90) (unit 1)
     (in_bom yes) (on_board yes) (dnp no)
-    (property "Reference" "C3" (at 148.59 89.535 90)
+    (property "Reference" "C3" (at 149.86 89.535 90)
       (effects (font (size 1.27 1.27)))
     )
-    (property "Value" "1uF" (at 147.955 92.075 90)
+    (property "Value" "1uF 50V" (at 147.32 92.075 90)
       (effects (font (size 1.27 1.27)))
     )
-    (property "Footprint" "RevK:C_0402" (at 154.94 89.8398 0)
+    (property "Footprint" "RevK:C_0402" (at 156.21 89.8398 0)
       (effects (font (size 1.27 1.27)) hide)
     )
-    (property "Datasheet" "~" (at 151.13 90.805 0)
+    (property "Datasheet" "~" (at 152.4 90.805 0)
       (effects (font (size 1.27 1.27)) hide)
     )
@@
       (effects (font (size 1.27 1.27)))
     )
-    (property "Value" "1uF" (at 138.43 137.795 90)
+    (property "Value" "1uF 50V" (at 136.525 137.795 90)
       (effects (font (size 1.27 1.27)))
     )
@@
     )
   )
-  (symbol (lib_id "Device:C") (at 151.13 95.885 90) (unit 1)
+  (symbol (lib_id "Device:C") (at 152.4 95.885 90) (unit 1)
     (in_bom yes) (on_board yes) (dnp no)
-    (property "Reference" "C3" (at 148.59 94.615 90)
+    (property "Reference" "C3" (at 149.86 94.615 90)
       (effects (font (size 1.27 1.27)))
     )
-    (property "Value" "1uF" (at 147.955 97.155 90)
+    (property "Value" "1uF 50V" (at 147.32 97.155 90)
       (effects (font (size 1.27 1.27)))
     )
-    (property "Footprint" "RevK:C_0402" (at 154.94 94.9198 0)
+    (property "Footprint" "RevK:C_0402" (at 156.21 94.9198 0)
       (effects (font (size 1.27 1.27)) hide)
     )
-    (property "Datasheet" "~" (at 151.13 95.885 0)
+    (property "Datasheet" "~" (at 152.4 95.885 0)
       (effects (font (size 1.27 1.27)) hide)
     )
@@
       (effects (font (size 1.27 1.27)))
     )
-    (property "Value" "1uF" (at 138.43 94.615 90)
+    (property "Value" "1uF 50V" (at 135.89 94.615 90)
       (effects (font (size 1.27 1.27)))
     )
@@
       (effects (font (size 1.27 1.27)))
     )
-    (property "Value" "100nF" (at 137.795 109.855 90)
+    (property "Value" "100nF 50V" (at 135.255 109.855 90)
       (effects (font (size 1.27 1.27)))
     )
@@
       (effects (font (size 1.27 1.27)))
     )
-    (property "Value" "1uF" (at 138.43 104.775 90)
+    (property "Value" "1uF 50V" (at 135.89 104.775 90)
       (effects (font (size 1.27 1.27)))
     )
@@
     )
   )
-  (symbol (lib_id "Device:C") (at 151.13 100.965 90) (unit 1)
+  (symbol (lib_id "Device:C") (at 152.4 100.965 90) (unit 1)
     (in_bom yes) (on_board yes) (dnp no)
-    (property "Reference" "C3" (at 147.955 99.695 90)
+    (property "Reference" "C3" (at 149.225 99.695 90)
       (effects (font (size 1.27 1.27)))
     )
-    (property "Value" "1uF" (at 147.955 102.235 90)
+    (property "Value" "1uF 50V" (at 147.32 102.235 90)
       (effects (font (size 1.27 1.27)))
     )
-    (property "Footprint" "RevK:C_0402" (at 154.94 99.9998 0)
+    (property "Footprint" "RevK:C_0402" (at 156.21 99.9998 0)
       (effects (font (size 1.27 1.27)) hide)
     )
-    (property "Datasheet" "~" (at 151.13 100.965 0)
+    (property "Datasheet" "~" (at 152.4 100.965 0)
       (effects (font (size 1.27 1.27)) hide)
     )
@@
       (effects (font (size 1.27 1.27)))
     )
-    (property "Value" "1uF" (at 138.43 99.695 90)
+    (property "Value" "1uF 50V" (at 135.89 99.695 90)
       (effects (font (size 1.27 1.27)))
     )
@@
       (effects (font (size 1.27 1.27)))
     )
-    (property "Value" "1uF" (at 138.43 89.535 90)
+    (property "Value" "1uF 50V" (at 136.525 89.535 90)
       (effects (font (size 1.27 1.27)))
     )
@@
       (effects (font (size 1.27 1.27)))
     )
-    (property "Value" "1uF" (at 148.59 140.335 90)
+    (property "Value" "1uF 50V" (at 146.05 140.335 90)
       (effects (font (size 1.27 1.27)))
     )
