File: PCB/EPD75/EPD75.kicad_pcb (KiCad board)
At the start: 2 copper layers, 35 parts, among them J1 Conn_01x26, J2 Shelly, J3 USB-PROG, Q1 DMG1012T, U3 MD8942, U4 ESP32-S3-MINI-1

Commit message: Started, but need a face up sockedt
Parts:
- J1: footprint RevK:24_Pins_0.5mm_Pitch_ZIF_Connector_UP -> RevK:HRS-FH12-24S-0.5SH-Face-Down
Connections:
- U4 pad 23: unconnected-(U4-GPIO19-Pad23) -> D-
- U4 pad 24: unconnected-(U4-GPIO20-Pad24) -> D+
- U4 pad 28: unconnected-(U4-GPIO33-Pad28) -> MOSI
- U4 pad 29: unconnected-(U4-GPIO34-Pad29) -> CLK
- U4 pad 31: unconnected-(U4-GPIO35-Pad31) -> CS
- U4 pad 32: unconnected-(U4-GPIO36-Pad32) -> DC
- U4 pad 33: unconnected-(U4-GPIO37-Pad33) -> RST
- U4 pad 34: unconnected-(U4-GPIO38-Pad34) -> BUSY

Commit message: Better connector
Parts:
- J1: footprint RevK:HRS-FH12-24S-0.5SH-Face-Down -> RevK:XUNPU-FPC-05FB-24PH20
- turned J1 to 180 degrees

Commit message: Needs tracking
Parts:
- added C19: 100nF, RevK:C_0402, F.Cu at (19.0, 46.6)
- added C21: 33pF, RevK:C_0402, F.Cu at (37.7, 109.7)
- added C22: 33pF, RevK:C_0402, F.Cu at (37.7, 111.5)
- added C23: 0.1uF, RevK:C_0402, F.Cu at (102.0, 72.0)
- added C24: 100nF, RevK:C_0402, F.Cu at (180.9, 46.5)
- added C25: 100nF, RevK:C_0402, F.Cu at (180.9, 153.4)
- added C26: 100nF, RevK:C_0402, F.Cu at (19.1, 153.4)
- added D10: XL-1010RGBC-WS2812B, RevK:SMD1010, F.Cu at (17.6, 153.4)
- added D4: XL-1010RGBC-WS2812B, RevK:SMD1010, F.Cu at (17.6, 46.6)
- added D5: XL-1010RGBC-WS2812B, RevK:SMD1010, F.Cu at (182.4, 46.6)
- added D6: D, RevK:D_SOD-123, F.Cu at (43.6, 99.1)
- added D7: BAV99S, RevK:SOT-363_SC-70-6, F.Cu at (31.1, 110.0)
- added D9: XL-1010RGBC-WS2812B, RevK:SMD1010, F.Cu at (182.4, 153.4)
- added J4: BTN1, RevK:PTSM-HH-2-RA-SMD, F.Cu at (153.0, 131.0)
- added J5: USB-C-Socket-V, RevK:USB-C-Socket-H, F.Cu at (100.0, 150.6)
- added J6: BTN2, RevK:PTSM-HH-2-RA-SMD, F.Cu at (152.0, 69.0)
- added J7: USB-C-Socket-V, RevK:USB-C-Socket-H, F.Cu at (179.6, 100.0)
- added J8: PWR, RevK:PTSM-HH-2-RA-SMD, F.Cu at (28.0, 133.0)
- added JP1: SolderJumper_3_Bridged12, RevK:SolderJumper3, F.Cu at (88.7, 71.5)
- added JP2: SolderJumper_3_Bridged12, RevK:SolderJumper3, F.Cu at (88.7, 75.0)
- added P1: 2, RevK:SolderPad, F.Cu at (149.0, 55.0)
- added P10: +, RevK:SolderPad, F.Cu at (155.0, 97.0)
- added P11: -, RevK:SolderPad, F.Cu at (155.0, 103.0)
- added P12: 5V, RevK:SolderPad, F.Cu at (155.0, 109.0)
- added P2: 1, RevK:SolderPad, F.Cu at (149.0, 145.0)
- added P3: -, RevK:SolderPad, F.Cu at (172.0, 145.0)
- added P4: -, RevK:SolderPad, F.Cu at (172.0, 55.0)
- added P5: 2, RevK:SolderPad, F.Cu at (155.0, 55.0)
- added P6: 1, RevK:SolderPad, F.Cu at (155.0, 145.0)
- added P7: +, RevK:SolderPad, F.Cu at (166.0, 145.0)
- added P8: +, RevK:SolderPad, F.Cu at (166.0, 55.0)
- added P9: GND, RevK:SolderPad, F.Cu at (155.0, 91.0)
- added R12: 5k1, RevK:R_0402, F.Cu at (98.2, 146.5)
- added R13: 5k1, RevK:R_0402, F.Cu at (102.3, 146.5)
- added R4: 5k1, RevK:R_0402, F.Cu at (175.7, 102.2)
- added R5: 5k1, RevK:R_0402, F.Cu at (175.6, 97.6)
- added R6: 100R, RevK:R_0402, F.Cu at (35.4, 109.8)
- added R7: 100R, RevK:R_0402, F.Cu at (35.4, 111.6)
- added R8: 3R, RevK:R_0402, F.Cu at (91.3, 75.0)
- C18: value 4.7uF -> 10uF
- moved U4 121.5 mm to (29.0, 100.0), turned to 90 degrees
- moved J2 119.4 mm to (23.9, 100.1), turned to -90 degrees
- moved C5 117.5 mm to (26.2, 109.0)
- moved C2 116.8 mm to (24.0, 109.0), turned to 180 degrees
- moved R3 114.1 mm to (25.5, 91.0), turned to 180 degrees
- moved C6 111.1 mm to (23.5, 91.0), turned to 180 degrees
- moved J3 109.1 mm to (33.9, 100.0), turned to 90 degrees
- moved C8 101.7 mm to (45.7, 100.6), turned to 90 degrees
- moved C10 98.1 mm to (48.2, 101.3)
- moved C9 96.4 mm to (50.7, 100.6), turned to 90 degrees
- moved R11 95.0 mm to (46.4, 97.4)
- moved R9 94.9 mm to (48.2, 97.4)
- moved R10 92.3 mm to (50.1, 97.4)
- moved U3 91.5 mm to (48.2, 99.3)
- moved L2 88.4 mm to (48.2, 103.9)
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Connections:
- J1 pad 8: GND -> Net-(J1-Pin_8)
- J3 pad 1: DC -> VBUS
- R1 pad 1: Net-(J1-Pin_3) -> Net-(JP2-A)
- R2 pad 1: Net-(J1-Pin_2) -> GND
- R2 pad 2: GND -> Net-(J1-Pin_2)
- U3 pad 5: DC -> PWR
- U4 pad 16: GND -> unconnected-(U4-GPIO12-Pad16)
- U4 pad 17: GND -> unconnected-(U4-GPIO13-Pad17)
- U4 pad 18: GND -> unconnected-(U4-GPIO14-Pad18)
- U4 pad 19: GND -> unconnected-(U4-GPIO15-Pad19)
- U4 pad 20: GND -> unconnected-(U4-GPIO16-Pad20)
- U4 pad 21: GND -> unconnected-(U4-GPIO17-Pad21)
- U4 pad 22: GND -> unconnected-(U4-GPIO18-Pad22)
- U4 pad 28: MOSI -> unconnected-(U4-GPIO33-Pad28)
- U4 pad 29: CLK -> RGB
- U4 pad 31: CS -> BUSY
- U4 pad 32: DC -> RST
- U4 pad 33: RST -> DC
- U4 pad 34: BUSY -> CS
- U4 pad 35: unconnected-(U4-GPIO39-Pad35) -> CLK
- U4 pad 36: unconnected-(U4-GPIO40-Pad36) -> MOSI
- U4 pad 37: unconnected-(U4-GPIO41-Pad37) -> BTN1
- U4 pad 38: unconnected-(U4-GPIO42-Pad38) -> BTN2
Routing:
- added copper zone on B.Cu, net GND
- added copper zone on F.Cu, net GND
Other:
- board outline added: 168 x 110 mm
- board text added: "+"
- board text added: "-"
- board text added: "1"
- board text added: "2"
- board text added: "34"
- board text added: "35"
- board text added: "36"
- board text added: "37"
- board text added: "38"
- board text added: "40"
- board text added: "41"
- board text added: "42"
- board text added: "A"
- board text added: "BTN1"
- board text added: "BTN2"
- board text added: "BUSY"
- board text added: "CLK"
- board text added: "CS"
- board text added: "DC"
- board text added: "MOSI"
- board text added: "RGB"
- board text added: "RST"
- board text added: "USB"
- board text added: "Waveshare 7.5{dblquote} EPD ESP32 Driver board"

Commit message: Initial tracking
Parts:
- removed C23: 0.1uF, RevK:C_0402
- moved C21 23.9 mm to (25.8, 88.9), turned to -90 degrees
- moved C22 23.5 mm to (31.4, 88.9), turned to 90 degrees
- moved R7 23.2 mm to (30.4, 88.9), turned to -90 degrees
- moved R6 22.6 mm to (26.7, 88.9), turned to 90 degrees
- moved D7 21.2 mm to (28.6, 89.0), turned to 90 degrees
- moved D3 7.20 mm to (100.5, 74.5), turned to 90 degrees
- moved D2 7.10 mm to (98.5, 74.5), turned to 90 degrees
- moved Q1 7.01 mm to (95.0, 70.2), turned to 90 degrees
- moved JP2 6.30 mm to (88.7, 68.7)
- moved R1 6.30 mm to (86.1, 68.7)
- moved R8 6.30 mm to (91.3, 68.7)
- moved C17 4.92 mm to (101.0, 71.7)
- moved L1 2.67 mm to (95.9, 72.9)
- moved C16 2.41 mm to (97.9, 70.2)
- moved R2 2.41 mm to (97.0, 70.2)
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Connections:
- P5 pad 1: Net-(J4-Pin_2) -> Net-(J6-Pin_2)
- P6 pad 1: Net-(J6-Pin_2) -> Net-(J4-Pin_2)
- R6 pad 1: Net-(J4-Pin_2) -> Net-(J6-Pin_2)
- R7 pad 1: Net-(J6-Pin_2) -> Net-(J4-Pin_2)
Routing:
- net +3.3V: track 0.00 -> 431.2 mm, vias 0 -> 9
- net PWR: track 0.00 -> 270.8 mm, vias 0 -> 4
- net VBUS: track 0.00 -> 204.3 mm, vias 0 -> 6
- net D+: track 0.00 -> 191.1 mm, vias 0 -> 2
- net D-: track 0.00 -> 190.4 mm
- net Net-(D4-O): track 0.00 -> 172.5 mm
- net Net-(D10-I): track 0.00 -> 165.7 mm, vias 0 -> 2
- net Net-(J4-Pin_2): track 0.00 -> 156.2 mm, vias 0 -> 2
- net Net-(J6-Pin_2): track 0.00 -> 150.0 mm, vias 0 -> 2
- net Net-(D5-O): track 0.00 -> 108.2 mm, vias 0 -> 2
- net MOSI: track 0.00 -> 88.9 mm
- net CLK: track 0.00 -> 87.2 mm
- net CS: track 0.00 -> 85.6 mm
- net DC: track 0.00 -> 83.9 mm
- net RST: track 0.00 -> 82.2 mm
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
Commit message: 50V caps
Parts:
- C1, C11, C12, C13, C15, C16, C3, C4, C7: value 1uF -> 1uF 50V
- C14: value 100nF -> 100nF 50V
Routing:
- net GND: vias 10 -> 12
Changed lines of the file:
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@@
         (effects (font (size 1 1) (thickness 0.15)))
     )
-    (fp_text value "100nF" (at 0 1.1 -90 unlocked) (layer "F.Fab") hide
+    (fp_text value "100nF 50V" (at 0 1.1 -90 unlocked) (layer "F.Fab") hide
         (effects (font (size 1 1) (thickness 0.15)))
     )
@@
         (effects (font (size 1 1) (thickness 0.15)))
     )
-    (fp_text value "1uF" (at 0 1.1 -90 unlocked) (layer "F.Fab") hide
+    (fp_text value "1uF 50V" (at 0 1.1 -90 unlocked) (layer "F.Fab") hide
         (effects (font (size 1 1) (thickness 0.15)))
     )
@@
         (effects (font (size 1 1) (thickness 0.15)))
     )
-    (fp_text value "1uF" (at 0 1.1 -90 unlocked) (layer "F.Fab") hide
+    (fp_text value "1uF 50V" (at 0 1.1 -90 unlocked) (layer "F.Fab") hide
         (effects (font (size 1 1) (thickness 0.15)))
     )
@@
         (effects (font (size 1 1) (thickness 0.15)))
     )
-    (fp_text value "1uF" (at 0 1.1 -90 unlocked) (layer "F.Fab") hide
+    (fp_text value "1uF 50V" (at 0 1.1 -90 unlocked) (layer "F.Fab") hide
         (effects (font (size 1 1) (thickness 0.15)))
     )
@@
         (effects (font (size 1 1) (thickness 0.15)))
     )
-    (fp_text value "1uF" (at 0 1.1 -90 unlocked) (layer "F.Fab") hide
+    (fp_text value "1uF 50V" (at 0 1.1 -90 unlocked) (layer "F.Fab") hide
         (effects (font (size 1 1) (thickness 0.15)))
     )
@@
         (effects (font (size 1 1) (thickness 0.15)))
     )
-    (fp_text value "1uF" (at 0 1.1 -90 unlocked) (layer "F.Fab") hide
+    (fp_text value "1uF 50V" (at 0 1.1 -90 unlocked) (layer "F.Fab") hide
         (effects (font (size 1 1) (thickness 0.15)))
     )
@@
         (effects (font (size 1 1) (thickness 0.15)))
     )
-    (fp_text value "1uF" (at 0 1.1 -90 unlocked) (layer "F.Fab") hide
+    (fp_text value "1uF 50V" (at 0 1.1 -90 unlocked) (layer "F.Fab") hide
         (effects (font (size 1 1) (thickness 0.15)))
     )
@@
         (effects (font (size 1 1) (thickness 0.15)))
     )
-    (fp_text value "1uF" (at 0 1.1 -90 unlocked) (layer "F.Fab") hide
+    (fp_text value "1uF 50V" (at 0 1.1 -90 unlocked) (layer "F.Fab") hide
         (effects (font (size 1 1) (thickness 0.15)))
     )
@@
         (effects (font (size 1 1) (thickness 0.15)))
     )
-    (fp_text value "1uF" (at 0 1.1 -90 unlocked) (layer "F.Fab") hide
+    (fp_text value "1uF 50V" (at 0 1.1 -90 unlocked) (layer "F.Fab") hide
         (effects (font (size 1 1) (thickness 0.15)))
     )
@@
         (effects (font (size 1 1) (thickness 0.15)))
     )
-    (fp_text value "1uF" (at 0 1.1 -90 unlocked) (layer "F.Fab") hide
+    (fp_text value "1uF 50V" (at 0 1.1 -90 unlocked) (layer "F.Fab") hide
         (effects (font (size 1 1) (thickness 0.15)))
     )
@@
   (segment (start 183.5 153.675) (end 183.5 147.7) (width 0.25) (layer "F.Cu") (net 1))
   (segment (start 16.6 153.775) (end 16.6 152.45) (width 0.25) (layer "F.Cu") (net 1))
+  (via (at 131.3 47.4) (size 0.8) (drill 0.4) (layers "F.Cu" "B.Cu") (free) (net 1))
   (via (at 93.2 71.7) (size 0.8) (drill 0.4) (layers "F.Cu" "B.Cu") (free) (net 1))
   (via (at 104.5 65.8) (size 0.8) (drill 0.4) (layers "F.Cu" "B.Cu") (free) (net 1))
   (via (at 103.5 71.8) (size 0.8) (drill 0.4) (layers "F.Cu" "B.Cu") (free) (net 1))
   (via (at 103.8 145.4) (size 0.8) (drill 0.4) (layers "F.Cu" "B.Cu") (free) (net 1))
+  (via (at 87.6 47) (size 0.8) (drill 0.4) (layers "F.Cu" "B.Cu") (free) (net 1))
   (via (at 93.3 67.4) (size 0.8) (drill 0.4) (layers "F.Cu" "B.Cu") (free) (net 1))
   (via (at 106.111371 72.113934) (size 0.8) (drill 0.4) (layers "F.Cu" "B.Cu") (free) (net 1))

Commit message: Checked
Parts:
- moved J2 14.7 mm to (34.8, 110.5), turned to 0 degrees
- moved J3 14.1 mm to (34.8, 114.0), turned to 0 degrees
- moved C1 2.00 mm to (105.8, 70.2)
- moved C11 2.00 mm to (102.2, 70.2)
- moved C12 2.00 mm to (101.3, 70.2)
- moved C13 2.00 mm to (100.4, 70.2)
- moved C14 2.00 mm to (99.5, 70.2)
- moved C15 2.00 mm to (96.8, 70.2)
- moved C16 2.00 mm to (95.9, 70.2)
- moved C17 2.00 mm to (99.0, 71.7)
- moved C18 2.00 mm to (98.6, 70.2)
- moved C3 2.00 mm to (104.9, 70.2)
- moved C4 2.00 mm to (104.0, 70.2)
- moved C7 2.00 mm to (103.1, 70.2)
- moved D1 2.00 mm to (100.6, 74.5)
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Routing:
- net VBUS: track 204.3 -> 237.9 mm, vias 6 -> 5
- net PWR: track 270.8 -> 291.5 mm
- net Net-(J2-Tx): track 4.66 -> 24.2 mm, vias 0 -> 1
- net D+: track 191.1 -> 207.4 mm, vias 2 -> 3
- net D-: track 190.4 -> 204.6 mm, vias 0 -> 1
- net Net-(J2-Rx): track 8.18 -> 19.8 mm, vias 0 -> 1
- net Net-(J2-0): track 5.15 -> 15.9 mm, vias 0 -> 1
- net RGB: track 65.7 -> 71.7 mm
- net GND: track 45.3 -> 47.8 mm, vias 12 -> 25
- net RST: track 82.2 -> 80.2 mm
- net MOSI: track 88.9 -> 86.9 mm
- net DC: track 83.9 -> 81.9 mm
- net CS: track 85.6 -> 83.6 mm
- net CLK: track 87.2 -> 85.2 mm
- net BUSY: track 80.5 -> 78.5 mm
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Other:
- outline, holes or cut-outs redrawn
- board text added: "0.47R"
- board text added: "3"
- board text added: "3R"
- board text added: "4"
- board text added: "www.me.uk"

Commit message: Silk
Other:
- board text added: "0R47"
- board text added: "B"
- board text added: "Made in China for Andrews & Arnold Ltd"
- board text added: "SPI"
- board text removed: "0.47R"
