File: PCB/EPD/EPD.kicad_sch (KiCad schematic)
At the start: 63 parts, among them J1 Conn_01x26, J2 Shelly, J3 USB-PROG, J4 BTN1, J6 BTN2, J7 USB-C-Socket-V, J8 PWR, P1 +, P10 2, P11 1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

Commit message: More general EPD driver
Connections:
- net BTN1: now also U2.6 (GPIO2); no longer U2.37 (GPIO41)
- net BTN2: now also U2.12 (GPIO8); no longer U2.38 (GPIO42)
- net BUSY: now also U2.38 (GPIO42); no longer U2.31 (GPIO35)
- net CLK: now also U2.34 (GPIO38); no longer U2.35 (GPIO39)
- net CS: now also U2.35 (GPIO39); no longer U2.34 (GPIO38)
- net DC: now also U2.36 (GPIO40); no longer U2.33 (GPIO37)
- net MOSI: now also U2.33 (GPIO37); no longer U2.36 (GPIO40)
- net RGB: now also U2.32 (GPIO36); no longer U2.29 (GPIO34)
- net RST: now also U2.37 (GPIO41); no longer U2.32 (GPIO36)
Changed lines of the file:
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@@
   (no_connect (at 48.895 83.82))
   (no_connect (at 48.895 71.12))
-  (no_connect (at 48.895 50.8))
+  (no_connect (at 79.375 68.58))
   (no_connect (at 119.38 146.685))
   (no_connect (at 48.895 68.58))
@@
   (no_connect (at 48.895 99.06))
   (no_connect (at 79.375 93.98))
-  (no_connect (at 48.895 66.04))
+  (no_connect (at 79.375 66.04))
   (no_connect (at 79.375 63.5))
   (no_connect (at 48.895 60.96))
@@
     )
   )
-  (global_label "BTN2" (shape input) (at 79.375 86.36 0) (fields_autoplaced)
-    (effects (font (size 1.27 1.27)) (justify left))
-    (property "Intersheetrefs" "${INTERSHEET_REFS}" (at 86.4836 86.36 0)
-      (effects (font (size 1.27 1.27)) (justify left) hide)
+  (global_label "BTN2" (shape input) (at 48.895 66.04 180) (fields_autoplaced)
+    (effects (font (size 1.27 1.27)) (justify right))
+    (property "Intersheetrefs" "${INTERSHEET_REFS}" (at 41.7864 66.04 0)
+      (effects (font (size 1.27 1.27)) (justify right) hide)
     )
   )
@@
     )
   )
-  (global_label "MOSI" (shape output) (at 79.375 81.28 0) (fields_autoplaced)
-    (effects (font (size 1.27 1.27)) (justify left))
-    (property "Intersheetrefs" "${INTERSHEET_REFS}" (at 86.3022 81.28 0)
+  (global_label "MOSI" (shape output) (at 79.375 73.66 0) (fields_autoplaced)
+    (effects (font (size 1.27 1.27)) (justify left))
+    (property "Intersheetrefs" "${INTERSHEET_REFS}" (at 86.3022 73.66 0)
       (effects (font (size 1.27 1.27)) (justify left) hide)
     )
@@
     )
   )
-  (global_label "BUSY" (shape output) (at 79.375 68.58 0) (fields_autoplaced)
-    (effects (font (size 1.27 1.27)) (justify left))
-    (property "Intersheetrefs" "${INTERSHEET_REFS}" (at 86.6046 68.58 0)
+  (global_label "BUSY" (shape output) (at 79.375 86.36 0) (fields_autoplaced)
+    (effects (font (size 1.27 1.27)) (justify left))
+    (property "Intersheetrefs" "${INTERSHEET_REFS}" (at 86.6046 86.36 0)
       (effects (font (size 1.27 1.27)) (justify left) hide)
     )
@@
     )
   )
-  (global_label "DC" (shape output) (at 79.375 73.66 0) (fields_autoplaced)
-    (effects (font (size 1.27 1.27)) (justify left))
-    (property "Intersheetrefs" "${INTERSHEET_REFS}" (at 84.246 73.66 0)
+  (global_label "DC" (shape output) (at 79.375 81.28 0) (fields_autoplaced)
+    (effects (font (size 1.27 1.27)) (justify left))
+    (property "Intersheetrefs" "${INTERSHEET_REFS}" (at 84.246 81.28 0)
       (effects (font (size 1.27 1.27)) (justify left) hide)
     )
@@
     )
   )
-  (global_label "RST" (shape output) (at 79.375 71.12 0) (fields_autoplaced)
-    (effects (font (size 1.27 1.27)) (justify left))
-    (property "Intersheetrefs" "${INTERSHEET_REFS}" (at 85.1531 71.12 0)
-      (effects (font (size 1.27 1.27)) (justify left) hide)
-    )
-  )
-  (global_label "CS" (shape output) (at 79.375 76.2 0) (fields_autoplaced)
-    (effects (font (size 1.27 1.27)) (justify left))
-    (property "Intersheetrefs" "${INTERSHEET_REFS}" (at 84.1855 76.2 0)
+  (global_label "RST" (shape output) (at 79.375 83.82 0) (fields_autoplaced)
+    (effects (font (size 1.27 1.27)) (justify left))
+    (property "Intersheetrefs" "${INTERSHEET_REFS}" (at 85.1531 83.82 0)
+      (effects (font (size 1.27 1.27)) (justify left) hide)
+    )
+  )
+  (global_label "CS" (shape output) (at 79.375 78.74 0) (fields_autoplaced)
+    (effects (font (size 1.27 1.27)) (justify left))
+    (property "Intersheetrefs" "${INTERSHEET_REFS}" (at 84.1855 78.74 0)
       (effects (font (size 1.27 1.27)) (justify left) hide)
     )
@@
     )
   )
-  (global_label "RGB" (shape output) (at 79.375 66.04 0) (fields_autoplaced)
-    (effects (font (size 1.27 1.27)) (justify left))
-    (property "Intersheetrefs" "${INTERSHEET_REFS}" (at 85.516 66.04 0)
+  (global_label "RGB" (shape output) (at 79.375 71.12 0) (fields_autoplaced)
+    (effects (font (size 1.27 1.27)) (justify left))
+    (property "Intersheetrefs" "${INTERSHEET_REFS}" (at 85.516 71.12 0)
       (effects (font (size 1.27 1.27)) (justify left) hide)
     )
@@
     )
   )
-  (global_label "CLK" (shape output) (at 79.375 78.74 0) (fields_autoplaced)
-    (effects (font (size 1.27 1.27)) (justify left))
-    (property "Intersheetrefs" "${INTERSHEET_REFS}" (at 85.2741 78.74 0)
+  (global_label "CLK" (shape output) (at 79.375 76.2 0) (fields_autoplaced)
+    (effects (font (size 1.27 1.27)) (justify left))
+    (property "Intersheetrefs" "${INTERSHEET_REFS}" (at 85.2741 76.2 0)
       (effects (font (size 1.27 1.27)) (justify left) hide)
     )
@@
     )
   )
-  (global_label "BTN1" (shape input) (at 79.375 83.82 0) (fields_autoplaced)
-    (effects (font (size 1.27 1.27)) (justify left))
-    (property "Intersheetrefs" "${INTERSHEET_REFS}" (at 86.4836 83.82 0)
-      (effects (font (size 1.27 1.27)) (justify left) hide)
-    )
-  )
+  (global_label "BTN1" (shape input) (at 48.895 50.8 180) (fields_autoplaced)
+    (effects (font (size 1.27 1.27)) (justify right))
+    (property "Intersheetrefs" "${INTERSHEET_REFS}" (at 41.7864 50.8 0)
+      (effects (font (size 1.27 1.27)) (justify right) hide)
+    )
+  )

Commit message: Panel
Parts:
- added PCB1: 70x70, RevK:PCB7070, symbol RevK:PCB
- added V1, V3, V4, V6: ~, RevK:VCUT70N, symbol RevK:VCUT
Changed lines of the file:
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@@
+    )
+  )
+  (symbol (lib_id "RevK:PCB") (at 274.32 173.355 0) (unit 1)
+    (in_bom no) (on_board yes) (dnp no)
+    (property "Reference" "PCB1" (at 274.32 183.515 0)
+      (effects (font (size 1.27 1.27)) hide)
+    )
+    (property "Value" "70x70" (at 274.32 173.355 0)
+      (effects (font (size 1.27 1.27)))
+    )
+    (property "Footprint" "RevK:PCB7070" (at 274.32 167.64 0)
+      (effects (font (size 1.27 1.27)) hide)
+    )
+    (property "Datasheet" "" (at 274.32 173.355 0)
+      (effects (font (size 1.27 1.27)) hide)
+    )
+    (instances
+      (project "EPD"
+        (path "/46c350bb-7de4-4e81-aafd-4af55e37aab0"
+          (reference "PCB1") (unit 1)
+        )
+      )
     )
   )
@@
     )
   )
+  (symbol (lib_id "RevK:VCUT") (at 274.32 175.895 0) (unit 1)
+    (in_bom no) (on_board yes) (dnp no) (fields_autoplaced)
+    (property "Reference" "V4" (at 274.32 174.625 0)
+      (effects (font (size 1.27 1.27)) hide)
+    )
+    (property "Value" "~" (at 274.32 175.895 0)
+      (effects (font (size 1.27 1.27)))
+    )
+    (property "Footprint" "RevK:VCUT70N" (at 274.32 177.165 0)
+      (effects (font (size 1.27 1.27)) hide)
+    )
+    (property "Datasheet" "" (at 274.32 175.895 0)
+      (effects (font (size 1.27 1.27)) hide)
+    )
+    (property "Sim.Enable" "0" (at 274.32 175.895 0)
+      (effects (font (size 1.27 1.27)) hide)
+    )
+    (instances
+      (project "EPD"
+        (path "/46c350bb-7de4-4e81-aafd-4af55e37aab0"
+          (reference "V4") (unit 1)
+        )
+      )
+    )
+  )
   (symbol (lib_id "power:GND") (at 255.27 29.845 0) (unit 1)
     (in_bom yes) (on_board yes) (dnp no)
@@
         (path "/46c350bb-7de4-4e81-aafd-4af55e37aab0"
           (reference "C2") (unit 1)
+        )
+      )
+    )
+  )
+  (symbol (lib_id "RevK:VCUT") (at 271.145 173.355 90) (unit 1)
+    (in_bom no) (on_board yes) (dnp no) (fields_autoplaced)
+    (property "Reference" "V1" (at 269.875 173.355 0)
+      (effects (font (size 1.27 1.27)) hide)
+    )
+    (property "Value" "~" (at 271.145 173.355 0)
+      (effects (font (size 1.27 1.27)))
+    )
+    (property "Footprint" "RevK:VCUT70N" (at 272.415 173.355 0)
+      (effects (font (size 1.27 1.27)) hide)
+    )
+    (property "Datasheet" "" (at 271.145 173.355 0)
+      (effects (font (size 1.27 1.27)) hide)
+    )
+    (property "Sim.Enable" "0" (at 271.145 173.355 0)
+      (effects (font (size 1.27 1.27)) hide)
+    )
+    (instances
+      (project "EPD"
+        (path "/46c350bb-7de4-4e81-aafd-4af55e37aab0"
+          (reference "V1") (unit 1)
+        )
+      )
+    )
+  )
+  (symbol (lib_id "RevK:VCUT") (at 277.495 173.355 90) (unit 1)
+    (in_bom no) (on_board yes) (dnp no) (fields_autoplaced)
+    (property "Reference" "V6" (at 276.225 173.355 0)
+      (effects (font (size 1.27 1.27)) hide)
+    )
+    (property "Value" "~" (at 277.495 173.355 0)
+      (effects (font (size 1.27 1.27)))
+    )
+    (property "Footprint" "RevK:VCUT70N" (at 278.765 173.355 0)
+      (effects (font (size 1.27 1.27)) hide)
+    )
+    (property "Datasheet" "" (at 277.495 173.355 0)
+      (effects (font (size 1.27 1.27)) hide)
+    )
+    (property "Sim.Enable" "0" (at 277.495 173.355 0)
+      (effects (font (size 1.27 1.27)) hide)
+    )
+    (instances
+      (project "EPD"
+        (path "/46c350bb-7de4-4e81-aafd-4af55e37aab0"
+          (reference "V6") (unit 1)
         )
       )
@@
         )
       )
+    )
+  )
+  (symbol (lib_id "RevK:VCUT") (at 274.32 170.815 0) (unit 1)
+    (in_bom no) (on_board yes) (dnp no) (fields_autoplaced)
+    (property "Reference" "V3" (at 274.32 169.545 0)
+      (effects (font (size 1.27 1.27)) hide)
+    )
+    (property "Value" "~" (at 274.32 170.815 0)
+      (effects (font (size 1.27 1.27)))
+    )
+    (property "Footprint" "RevK:VCUT70N" (at 274.32 172.085 0)
+      (effects (font (size 1.27 1.27)) hide)
+    )
+    (property "Datasheet" "" (at 274.32 170.815 0)
+      (effects (font (size 1.27 1.27)) hide)
+    )
+    (property "Sim.Enable" "0" (at 274.32 170.815 0)
+      (effects (font (size 1.27 1.27)) hide)
+    )
+    (instances
+      (project "EPD"
+        (path "/46c350bb-7de4-4e81-aafd-4af55e37aab0"
+          (reference "V3") (unit 1)
+        )
+      )
